File: PCB/Porsche_Panamera/Porsche_Panamera.kicad_sch (KiCad schematic)
At the start: 0 parts

Commit message: Datenblatt IP5306 ergaenzt und Schaltplan erweitert
Parts:
- added C1, C2: C, symbol Device:C
- added D1, D10, D11, D12, D13: LED, symbol Device:LED
- added D2, D3, D4, D5, D6, D7, D8, D9: D, Diode_THT:D_DO-35_SOD27_P7.62mm_Horizontal, symbol Device:D
- added M1: Motor_Servo, Package_SON:WSON-8-1EP_6x5mm_P1.27mm_EP3.4x4mm, symbol Motor:Motor_Servo
- added M2: Motor_DC, symbol Motor:Motor_DC
- added R1: 1000, Package_TO_SOT_SMD:TO-252-2, symbol Device:R
- added U1: ESP32-C3-WROOM-02, RF_Module:ESP32-C3-WROOM-02, symbol RF_Module:ESP32-C3-WROOM-02
- added U2: L298N, Package_TO_SOT_THT:TO-220-15_P2.54x5.08mm_StaggerOdd_Lead4.58mm_Vertical, symbol Driver_Motor:L298N
- added U3: KA78M05_TO252, Package_TO_SOT_SMD:TO-252-2, symbol Regulator_Linear:KA78M05_TO252
- added U4: IP5306, lcsc_footprints:C181692_ESOP-8_L4_9-W3_9-P1_27-LS6_0-BL-EP, symbol lcsc_imported:IP5306
Connections:
- new net: U1.19 (GND), U1.9 (GND)
- new net: U1.3 (IO4), U2.5 (IN1)
- new net: U1.4 (IO5), U2.7 (IN2)
- new net: C1.2, C2.1, D1.1 (K), D2.1 (K), D3.1 (K), D4.1 (K), D5.1 (K), U2.4 (Vs)
- new net: D2.2 (A), D6.1 (K), M2.1 (+), U2.2 (OUT1)
- new net: D4.2 (A), D8.1 (K)
- new net: D5.2 (A), D9.1 (K)
- new net: C1.1, R1.1, U3.3 (VO)
- new net: D1.2 (A), R1.2
- new net: U2.9 (Vss), U3.1 (VI)
- new net: D3.2 (A), D7.1 (K), M2.2 (-), U2.3 (OUT2)
- new net GNDREF: C2.2, D6.2 (A), D7.2 (A), D8.2 (A), D9.2 (A), U2.1 (SENSE_A), U2.15 (SENSE_B), U2.8 (GND), U3.2 (GND), U4.9 (EP)

Commit message: Schaltplan weiter bearbeitet, Schaltung um IP5306
Parts:
- added C3, C4: 10uF, symbol Device:C
- added D14: LED, symbol Device:LED
- added L1: 20u, Package_SO:SOIC-28W_7.5x17.9mm_P1.27mm, symbol Device:L
- added R2: 2, Package_TO_SOT_SMD:TO-252-2, symbol Device:R
- added R3: 20, Package_TO_SOT_SMD:TO-252-2, symbol Device:R
- added R4: 10000, Package_TO_SOT_SMD:TO-252-2, symbol Device:R
- added SW1: SW_DPST_x2, Button_Switch_SMD:Nidec_Copal_CAS-120A, symbol Switch:SW_DPST_x2
Connections:
- net GNDREF: now also M1.3 (-), U1.19 (GND), U1.9 (GND), C3.2, C4.2, D14.1 (K), SW1.2 (B)
- net at D13.1 (K): now also D10.2 (A), U4.2 (LED1)
- net at D13.2 (A): now also D10.1 (K), D11.1 (K), D12.2 (A), U4.4 (LED3)
- net at D12.1 (K): now also D11.2 (A), U4.3 (LED2)
- net at U4.5 (KEY): now also R3.1, R4.1
- net at U4.6 (BAT): now also C3.1, L1.2, R2.1
- net at U4.7 (SW): now also L1.1
- new net: D14.2 (A), R3.2
- new net: C4.1, R2.2
- new net: R4.2, SW1.1 (A)
